File: Neo7m_eval_board.sch (EAGLE design)
At the start: 18 parts, among them CON4 U.FL, IC1 MC33269D-3.3

Commit message: Update, connected both DC jack ground connections to ground
Connections:
- net GND: now also VIN_5V_TO_12V.GND1
Changed lines of the file:
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@@
 <setting verticaltext="up"/>
 </settings>
-<grid distance="0.1" unitdist="inch" unit="inch" style="lines" multiple="1" display="no" altdistance="0.01" altunitdist="inch" altunit="inch"/>
+<grid distance="0.05" unitdist="inch" unit="inch" style="lines" multiple="1" display="no" altdistance="0.01" altunitdist="inch" altunit="inch"/>
 <layers>
 <layer number="1" name="Top" color="4" fill="1" visible="no" active="no"/>
@@
 <junction x="-203.2" y="-53.34"/>
 <pinref part="GND" gate="1" pin="GND"/>
-<pinref part="VIN_5V_TO_12V" gate="DCJACK" pin="GND2"/>
-<wire x1="-347.98" y1="-38.1" x2="-347.98" y2="-60.96" width="0.1524" layer="91"/>
 <pinref part="N3" gate="P1" pin="S"/>
-<wire x1="-350.52" y1="-60.96" x2="-347.98" y2="-60.96" width="0.1524" layer="91"/>
 <pinref part="IC1" gate="G$1" pin="ADJ"/>
 <wire x1="-284.48" y1="-53.34" x2="-284.48" y2="-50.8" width="0.1524" layer="91"/>
@@
 <wire x1="-304.8" y1="-53.34" x2="-284.48" y2="-53.34" width="0.1524" layer="91"/>
 <junction x="-304.8" y="-53.34"/>
+<wire x1="-350.52" y1="-60.96" x2="-347.98" y2="-60.96" width="0.1524" layer="91"/>
 <wire x1="-347.98" y1="-60.96" x2="-284.48" y2="-60.96" width="0.1524" layer="91"/>
 <wire x1="-284.48" y1="-60.96" x2="-284.48" y2="-53.34" width="0.1524" layer="91"/>
@@
 <wire x1="-134.62" y1="-48.26" x2="-121.92" y2="-48.26" width="0.1524" layer="91"/>
 <wire x1="-121.92" y1="-48.26" x2="-121.92" y2="-66.04" width="0.1524" layer="91"/>
-<junction x="-347.98" y="-60.96"/>
 <junction x="-284.48" y="-53.34"/>
 <junction x="-254" y="-53.34"/>
@@
 <wire x1="-139.7" y1="-22.86" x2="-106.68" y2="-22.86" width="0.1524" layer="91"/>
 <junction x="-139.7" y="-22.86"/>
-</segment>
-<segment>
+<pinref part="VIN_5V_TO_12V" gate="DCJACK" pin="GND2"/>
+<pinref part="VIN_5V_TO_12V" gate="DCJACK" pin="GND1"/>
+<wire x1="-347.98" y1="-38.1" x2="-347.98" y2="-41.91" width="0.1524" layer="91"/>
+<wire x1="-347.98" y1="-41.91" x2="-347.98" y2="-60.96" width="0.1524" layer="91"/>
+<junction x="-347.98" y="-41.91"/>
+<junction x="-347.98" y="-60.96"/>
+</segment>
+<segment>
