File: Neo7m_eval_board.brd (EAGLE design)
At the start: 55.1 x 46.7 mm, 18 parts, among them CON4 U.FL, IC1 MC33269D-3.3

Commit message: Update Neo7m_eval_board.brd
Connections:
- net GND: now also VIN_5V_TO_12V.GND1
Changed lines of the file:
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@@
 <description language="de">&lt;b&gt;EAGLE Design Rules&lt;/b&gt;
 &lt;p&gt;
-Die Standard-Design-Rules sind so gewÃ¤hlt, dass sie fÃ¼r
+Die Standard-Design-Rules sind so gewählt, dass sie für
 die meisten Anwendungen passen. Sollte ihre Platine
 besondere Anforderungen haben, treffen Sie die erforderlichen
@@
 <contactref element="C13" pad="2"/>
 <contactref element="C14" pad="2"/>
-<contactref element="VIN_5V_TO_12V" pad="GND2"/>
 <contactref element="N3" pad="P1"/>
 <contactref element="IC1" pad="1"/>
@@
 <contactref element="U$1" pad="G2"/>
 <contactref element="U$1" pad="G1"/>
+<contactref element="VIN_5V_TO_12V" pad="GND2"/>
+<contactref element="VIN_5V_TO_12V" pad="GND1"/>
 </signal>
 <signal name="+3V3">
